Commit message: New files added and some fixes

File: kuka_control/models/car_door/car_door.urdf.xacro (robot description, xacro)
@@ -6,5 +6,5 @@
   <!-- Car door (Vito) -->
   <xacro:car_door name="door1" parent="base_link">
-      <origin xyz="0.0 0.0 0.6" rpy="0 0 0" />
+      <origin xyz="0.0 0.0 0.8" rpy="0 0 0" />
   </xacro:car_door>
 </robot>

File: kuka_control/models/car_door/car_door.xacro (robot description, xacro)
@@ -12,4 +12,9 @@
           <mesh filename="package://kuka_control/models/car_door/meshes/door_vito.stl"/>
         </geometry>
+        <!--
+        <material name="red">
+        	<color rgba="1 0 0 1"/>
+        </material>
+        -->
       </visual>
       <collision name="collision">
@@ -24,4 +29,9 @@
       <child link="${name}"/>
   </joint>
+<!--
+  <gazebo reference="${name}">
+    <material>Gazebo/Orange</material>
+  </gazebo>
+-->
   </xacro:macro>
 </robot>

File: kuka_description/urdf/kr6r900sixx.urdf.xacro (robot description, xacro)
@@ -6,4 +6,10 @@
     <xacro:include filename="$(find kuka_description)/urdf/kr6r900sixx.gazebo.xacro" />
   </xacro:if>
+  <!-- Include Kuka KR6 model -->
   <xacro:include filename="$(find kuka_description)/urdf/kr6r900sixx.xacro" />
+  <!-- Include the force-torque-sensor model -->
+  <xacro:include filename="$(find sensor_description)/urdf/ft_sensor_ati.urdf.xacro"/>
+  <xacro:ft_sensor_axia80 parent="tool0" name="axia80" type="axia80">
+    <origin xyz="0 0 0.015" rpy="0 0 0"/>
+  </xacro:ft_sensor_axia80>
 </robot>
