Commit message: FT-sensor, tool and door xacro files added

File: kuka_control/models/ft_sensor/ft_sensor.urdf.xacro (robot description, xacro)
@@ -2,6 +2,6 @@
 <robot xmlns:xacro="http://ros.org/wiki/xacro" name="ft_sensor">
     <!-- Include all available models -->
-    <xacro:include filename="$(find kuka_control)/urdf/models.urdf.xacro"/>
-    <xacro:include filename="$(find kuka_control)/urdf/ft_sensor.gazebo.xacro"/>
+    <xacro:include filename="$(find kuka_control)/models/ft_sensor/models.urdf.xacro"/>
+    <xacro:include filename="$(find kuka_control)/models/ft_sensor/ft_sensor.gazebo.xacro"/>
     <!-- Base model for all sensor to have common frame names -->
     <xacro:macro name="ft_sensor" params="parent name type *origin">

File: kuka_control/models/ft_sensor/ft_sensor_ati.urdf.xacro (robot description, xacro)
@@ -2,7 +2,7 @@
 <robot xmlns:xacro="http://ros.org/wiki/xacro" name="ft_sensor_ati">
     <!-- Include all available models -->
-    <xacro:include filename="$(find kuka_control)/urdf/models.urdf.xacro"/>
-    <!--<xacro:include filename="$(find kuka_control)/urdf/ft_sensor.gazebo.xacro"/>-->
-    <xacro:include filename="$(find kuka_control)/urdf/ft_sensor_ati.gazebo.xacro"/>
+    <xacro:include filename="$(find kuka_control)/models/ft_sensor/models.urdf.xacro"/>
+    <!--<xacro:include filename="$(find kuka_control)/models/ft_sensor/ft_sensor.gazebo.xacro"/>-->
+    <xacro:include filename="$(find kuka_control)/models/ft_sensor/ft_sensor_ati.gazebo.xacro"/>
     <!-- Base model for all sensor to have common frame names -->
     <xacro:macro name="ft_sensor_nano17" params="parent name type *origin">

File: kuka_control/models/ft_sensor/models.urdf.xacro (robot description, xacro)
@@ -30,5 +30,5 @@
 				<geometry>
 					<!-- cylinder radius="0.0085" length="0.0145"/ -->
-					<mesh filename="package://kuka_control/meshes/nano17a.stl"/>
+					<mesh filename="package://kuka_control/models/ft_sensor/meshes/nano17a.stl"/>
 				</geometry>
 			</visual>
@@ -74,5 +74,5 @@
 			<geometry>
 				<!-- <cylinder radius="0.041" length="0.025"/> -->
-				<mesh filename="package://kuka_control/meshes/axia80.dae"/>
+				<mesh filename="package://kuka_control/models/ft_sensor/meshes/axia80.dae"/>
 			</geometry>
 		</visual>
@@ -120,5 +120,5 @@
 			<origin xyz="0 0 0" rpy="0 0 0"/>
 			<geometry>
-				<mesh filename="package://kuka_control/meshes/mini45.dae"/>
+				<mesh filename="package://kuka_control/models/ft_sensor/meshes/mini45.dae"/>
 			</geometry>
 		</visual>
@@ -162,5 +162,5 @@
 			<origin xyz="0 0 0.0134" rpy="${M_PI} 0 ${M_PI/2}"/>
 			<geometry>
-				<mesh filename="package://kuka_control/meshes/ftsensor45a.dae"/>
+				<mesh filename="package://kuka_control/models/ft_sensor/meshes/ftsensor45a.dae"/>
 			</geometry>
 		</visual>

File: kuka_description/urdf/kr6r900sixx.urdf.xacro (robot description, xacro)
@@ -9,7 +9,12 @@
   <xacro:include filename="$(find kuka_description)/urdf/kr6r900sixx.xacro" />
   <!-- Include the force-torque-sensor model -->
-  <xacro:include filename="$(find sensor_description)/urdf/ft_sensor_ati.urdf.xacro"/>
+  <xacro:include filename="$(find kuka_control)/models/ft_sensor/ft_sensor_ati.urdf.xacro"/>
   <xacro:ft_sensor_axia80 parent="tool0" name="axia80" type="axia80">
     <origin xyz="0 0 0.015" rpy="0 0 0"/>
   </xacro:ft_sensor_axia80>
+  <!-- Include tool model -->
+  <xacro:include filename="$(find kuka_control)/models/tool/tool.urdf.xacro"/>
+  <xacro:tool parent="axia80_ft_measure" name="tool1">
+    <origin xyz="0 0 0.013" rpy="0 0 0"/>
+  </xacro:tool>
 </robot>
