Commit message: Two new packages and some xacro and DAE files added.

File: kuka_control/models/brida/brida.urdf.xacro (robot description, xacro)
@@ -2,8 +2,8 @@
 <robot name="cell" xmlns:xacro="http://ros.org/wiki/xacro">
   <xacro:arg name="gazebo" default="false"/>
-  <!-- Tool -->
-  <xacro:include filename="$(find kuka_control)/models/tool/tool.xacro" />
-  <xacro:tool name="tool" parent="base_link">
+  <!-- Brida -->
+  <xacro:include filename="$(find kuka_control)/models/brida/brida.xacro" />
+  <xacro:brida name="brida" parent="tool0">
       <origin xyz="0.0 0.0 0.0" rpy="0 0 0" />
-  </xacro:tool>
+  </xacro:brida>
 </robot>

File: kuka_control/models/ft_sensor/ft_sensor_ati.urdf.xacro (robot description, xacro)
@@ -75,4 +75,34 @@
     </xacro:macro>
     <!-- Base model for all sensor to have common frame names -->
+    <xacro:macro name="ft_sensor_axia80_real" params="parent name type *origin">
+    <joint name="${name}_base_joint" type="fixed">
+	<xacro:insert_block name="origin"/>
+	<parent link="${parent}"/>
+	<child link="${name}_ft_base"/>
+    </joint>
+    <link name="${name}_ft_base">
+	<xacro:insert_block name="axia80"/>
+    </link>
+    <joint name="${name}_measure_joint" type="fixed">
+	<xacro:insert_block name="axia80_measure_frame"/>
+	<parent link="${name}_ft_base"/>
+	<child link="${name}_ft_measure"/>
+    </joint>
+    <link name="${name}_ft_measure">
+        <xacro:insert_block name="axia80_platform"/>
+    </link>
+    <transmission name="${name}_tran_ft">
+      <type>transmission_interface/SimpleTransmission</type>
+      <joint name="${name}_measure_joint">
+        <hardwareInterface>hardware_interface/EffortJointInterface</hardwareInterface>
+      </joint>
+      <actuator name="${name}_motor_ft">
+        <hardwareInterface>hardware_interface/EffortJointInterface</hardwareInterface>
+        <mechanicalReduction>1</mechanicalReduction>
+      </actuator>
+    </transmission>
+    <xacro:ft_sensor_gazebo name="${name}" parent="${parent}" type="${type}"/>
+    </xacro:macro>
+    <!-- Base model for all sensor to have common frame names -->
     <xacro:macro name="ft_sensor_mini45" params="parent name type *origin">
     <joint name="${name}_base_joint" type="fixed">

File: kuka_control/models/ft_sensor/models.urdf.xacro (robot description, xacro)
@@ -67,7 +67,7 @@
 		<inertial>
 			<!--<mass value="0.3"/>-->
-			<mass value="0.01"/>
+			<mass value="0.00001"/>
 			<origin xyz="0 0 0.0125"  />
-			<xacro:cylinder_inertia_def radius="0.041" length="0.025" mass="0.01"/>
+			<xacro:cylinder_inertia_def radius="0.041" length="0.025" mass="0.00001"/>
 		</inertial>
 		<visual>
@@ -87,7 +87,7 @@
 	<xacro:property name="axia80_platform">
 		<inertial>
-			<mass value="0.005"/>
+			<mass value="0.00001"/>
 			<origin xyz="0 0 0.0125"  />
-			<xacro:cylinder_inertia_def radius="0.041" length="0.005" mass="0.005"/>
+			<xacro:cylinder_inertia_def radius="0.041" length="0.005" mass="0.00001"/>
 		</inertial>
 		<!--<visual>

File: kuka_control/models/sensors/asus_camera.urdf.xacro (robot description, xacro)
@@ -75,5 +75,5 @@
       <gazebo reference="${name}_depth_frame">
         <sensor type="depth" name="${name}">
-          <update_rate>5</update_rate>
+          <update_rate>30</update_rate>
           <camera>
             <horizontal_fov>${62.8 * M_PI/180.0}</horizontal_fov>

File: kuka_control/models/sensors/kinect_camera.urdf.xacro (robot description, xacro)
@@ -58,13 +58,15 @@
       <gazebo reference="${name}_depth_frame">
         <sensor type="depth" name="${name}">
-          <update_rate>5</update_rate>
+          <update_rate>30</update_rate>
           <camera>
             <horizontal_fov>${60 * M_PI/180.0}</horizontal_fov>
             <image>
               <format>B8G8R8</format>
-              <width>640</width>
-              <height>480</height>
+              <!--<width>640</width>
+              <height>480</height>-->
               <!--<width>320</width>
               <height>240</height>-->
+              <width>160</width>
+              <height>120</height>
             </image>
             <clip>

File: kuka_control/models/tool/tool.xacro (robot description, xacro)
@@ -1,5 +1,18 @@
 <?xml version="1.0"?>
 <robot xmlns:xacro="http://ros.org/wiki/xacro">
+    <!-- Common tools: PI, inertias of a cuboid and cylinder -->
     <xacro:property name="M_PI" value="3.1415926535897931" />
+    <xacro:macro name="cuboid_inertia_def" params="width height length mass">
+    <inertia ixx="${mass * (height * height + length * length) / 12}"
+	     iyy="${mass * (width * width + length * length) / 12}"
+	     izz="${mass * (width * width + height * height) / 12}"
+	     ixy="0" iyz="0" ixz="0"/>
+    </xacro:macro>
+    <xacro:macro name="cylinder_inertia_def" params="radius length mass">
+    <inertia ixx="${mass * radius* radius / 2}"
+	     iyy="${mass * radius* radius / 2}"
+	     izz="${mass * (3 * radius * radius + length * length) / 12}"
+	     ixy="0" iyz="0" ixz="0"/>
+    </xacro:macro>
     <xacro:macro name="tool" params="name parent *origin">
       <joint name="${name}_base_joint" type="fixed">
@@ -29,7 +42,8 @@
       <link name="${name}_base">
         <inertial>
-          <mass value="0.005" />
+          <mass value="0.00001" />
           <origin xyz="0 0 0" rpy="0 0 0" />
-          <inertia ixx="0.0001" ixy="0" ixz="0" iyy="0.0001" iyz="0" izz="0.0001" />
+          <!--<inertia ixx="0.0001" ixy="0" ixz="0" iyy="0.0001" iyz="0" izz="0.0001" />-->
+	  <xacro:cylinder_inertia_def radius="0.0325" length="0.09" mass="0.00001"/>
         </inertial>
         <visual>
@@ -53,7 +67,8 @@
       <link name="${name}_tip">
         <inertial>
-          <mass value="0.0005" />
+          <mass value="0.00001" />
           <origin xyz="0 0 0" rpy="0 0 0" />
-          <inertia ixx="0.00001" ixy="0" ixz="0" iyy="0.00001" iyz="0" izz="0.00001" />
+          <!--<inertia ixx="0.00001" ixy="0" ixz="0" iyy="0.00001" iyz="0" izz="0.00001" />-->
+	  <xacro:cylinder_inertia_def radius="0.005" length="0.01" mass="0.00001"/>
         </inertial>
         <visual>

File: kuka_description/urdf/kr6r900sixx.urdf.xacro (robot description, xacro)
@@ -8,13 +8,5 @@
   <!-- Include Kuka KR6 model -->
   <xacro:include filename="$(find kuka_description)/urdf/kr6r900sixx.xacro" />
-  <!-- Include the force-torque-sensor model -->
-  <xacro:include filename="$(find kuka_control)/models/ft_sensor/ft_sensor_ati.urdf.xacro"/>
-  <xacro:ft_sensor_axia80 parent="tool0" name="axia80" type="axia80">
-    <origin xyz="0 0 0.015" rpy="0 0 0"/>
-  </xacro:ft_sensor_axia80>
-  <!-- Include tool model -->
-  <xacro:include filename="$(find kuka_control)/models/tool/tool.urdf.xacro"/>
-  <xacro:tool parent="axia80_ft_measure" name="tool1">
-    <origin xyz="0 0 0.013" rpy="0 0 0"/>
-  </xacro:tool>
+  <!-- Include FT-sensor and tool -->
+  <xacro:include filename="$(find kuka_control)/models/ft_tool.xacro" />
 </robot>
