Commit message: pykdl updated for teleoperation with gamepad

File: kuka_control/models/brida/brida.xacro (robot description, xacro)
@@ -23,8 +23,8 @@
       <link name="${name}_link">
         <inertial>
-          <mass value="0.00001" />
+          <mass value="0.05" />
           <origin xyz="0 0 0" rpy="0 0 0" />
           <!--<inertia ixx="0.0001" ixy="0" ixz="0" iyy="0.0001" iyz="0" izz="0.0001" />-->
-	  <xacro:cylinder_inertia_def radius="0.025" length="0.019" mass="0.00001"/>
+	  <xacro:cylinder_inertia_def radius="0.025" length="0.019" mass="0.05"/>
         </inertial>
         <visual>

File: kuka_control/models/ft_sensor/models.urdf.xacro (robot description, xacro)
@@ -67,7 +67,7 @@
 		<inertial>
 			<!--<mass value="0.3"/>-->
-			<mass value="0.00001"/>
+			<mass value="0.25"/>
 			<origin xyz="0 0 0.0125"  />
-			<xacro:cylinder_inertia_def radius="0.041" length="0.025" mass="0.00001"/>
+			<xacro:cylinder_inertia_def radius="0.041" length="0.025" mass="0.25"/>
 		</inertial>
 		<visual>
@@ -87,7 +87,7 @@
 	<xacro:property name="axia80_platform">
 		<inertial>
-			<mass value="0.00001"/>
+			<mass value="0.05"/>
 			<origin xyz="0 0 0.0125"  />
-			<xacro:cylinder_inertia_def radius="0.041" length="0.005" mass="0.00001"/>
+			<xacro:cylinder_inertia_def radius="0.041" length="0.005" mass="0.05"/>
 		</inertial>
 		<!--<visual>

File: kuka_control/models/tool/tool.xacro (robot description, xacro)
@@ -42,8 +42,8 @@
       <link name="${name}_base">
         <inertial>
-          <mass value="0.00001" />
+          <mass value="0.2" />
           <origin xyz="0 0 0" rpy="0 0 0" />
           <!--<inertia ixx="0.0001" ixy="0" ixz="0" iyy="0.0001" iyz="0" izz="0.0001" />-->
-	  <xacro:cylinder_inertia_def radius="0.0325" length="0.09" mass="0.00001"/>
+          <xacro:cylinder_inertia_def radius="0.0325" length="0.09" mass="0.2"/>
         </inertial>
         <visual>
@@ -67,8 +67,8 @@
       <link name="${name}_tip">
         <inertial>
-          <mass value="0.00001" />
+          <mass value="0.001" />
           <origin xyz="0 0 0" rpy="0 0 0" />
           <!--<inertia ixx="0.00001" ixy="0" ixz="0" iyy="0.00001" iyz="0" izz="0.00001" />-->
-	  <xacro:cylinder_inertia_def radius="0.005" length="0.01" mass="0.00001"/>
+          <xacro:cylinder_inertia_def radius="0.005" length="0.01" mass="0.001"/>
         </inertial>
         <visual>
@@ -90,5 +90,5 @@
         <mu1 value="0.01" />
         <mu2 value="0.01" />
-        <kp  value="100" />
+        <kp  value="10000" />
         <kd  value="0.1" />
         <material>Gazebo/Grey</material>

File: kuka_description/urdf/kr6r900sixx_macro.xacro (robot description, xacro)
@@ -10,5 +10,6 @@
   <xacro:property name="mass4" value="1.7" />
   <xacro:property name="mass5" value="0.7" />
-  <xacro:property name="mass6" value="0.05" />
+<!--  <xacro:property name="mass6" value="0.05" />-->
+  <xacro:property name="mass6" value="1.0" />
   <xacro:property name="length0" value="0.215" />
   <xacro:property name="length1" value="0.26" />
@@ -17,5 +18,6 @@
   <xacro:property name="length4" value="0.34" />
   <xacro:property name="length5" value="0.08" />
-  <xacro:property name="length6" value="0.008" />
+<!--  <xacro:property name="length6" value="0.008" />-->
+  <xacro:property name="length6" value="0.021" />
   <xacro:property name="diameter0" value="0.2" />
   <xacro:property name="diameter1" value="0.2" />
