Commit message: PID control updated. Cell mass increased. Rviz config changed.

File: kuka_control/models/cell/cell.xacro (robot description, xacro)
@@ -4,5 +4,5 @@
   <link name="base">
       <inertial>
-          <mass value="100" />
+          <mass value="500" />
           <origin xyz="0 0 0" rpy="0 0 0" />
           <inertia ixx="1" ixy="0" ixz="0" iyy="1" iyz="0" izz="1" />

File: kuka_control/models/tool/tool.xacro (robot description, xacro)
@@ -88,7 +88,7 @@
         <turnGravityOff>true</turnGravityOff>
         <selfCollide>true</selfCollide>
-        <mu1 value="0.01" />
-        <mu2 value="0.01" />
-        <kp  value="10000" />
+        <mu1 value="1" />
+        <mu2 value="1" />
+        <kp  value="1000000" />
         <kd  value="0.1" />
         <material>Gazebo/Grey</material>
