Commit message: New media and models folders added. Gamepad teleoperation with up-down joint switch.

File: kuka_control/models/cell/cell.urdf.xacro (robot description, xacro)
@@ -7,4 +7,5 @@
   <xacro:include filename="$(find kuka_control)/models/sensors/camera.urdf.xacro" />
   <!-- Car door -->
-  <xacro:include filename="$(find kuka_control)/models/car_door/car_door.urdf.xacro" />
+<!--  <xacro:include filename="$(find kuka_control)/models/car_door/car_door.urdf.xacro" />-->
+  <xacro:include filename="$(find kuka_control)/models/box/box.urdf.xacro" />
 </robot>

File: kuka_control/models/cell/cell.xacro (robot description, xacro)
@@ -1,6 +1,7 @@
 <?xml version="1.0" ?>
 <robot name="cell" xmlns:xacro="http://ros.org/wiki/xacro">
-  <link name="base_link"/>
-  <link name="base">
+  <!-- World frame (for Gazebo) -->
+  <link name="world"/>
+  <link name="base_link">
       <inertial>
           <mass value="500" />
@@ -19,8 +20,12 @@
       </collision>
   </link>
+  <!-- Cell fixed to world frame  -->
   <joint name="base_joint" type="fixed">
       <origin xyz="0.0 0.0 0.0" rpy="0 0 0" />
-      <parent link="base_link" />
-      <child link="base"/>
+      <parent link="world" />
+      <child link="base_link"/>
   </joint>
+  <gazebo>
+    <static>true</static>
+  </gazebo>
 </robot>

File: kuka_control/models/tool/tool.xacro (robot description, xacro)
@@ -1,18 +1,5 @@
 <?xml version="1.0"?>
 <robot xmlns:xacro="http://ros.org/wiki/xacro">
-    <!-- Common tools: PI, inertias of a cuboid and cylinder -->
-    <xacro:property name="M_PI" value="3.1415926535897931" />
-    <xacro:macro name="cuboid_inertia_def" params="width height length mass">
-    <inertia ixx="${mass * (height * height + length * length) / 12}"
-	     iyy="${mass * (width * width + length * length) / 12}"
-	     izz="${mass * (width * width + height * height) / 12}"
-	     ixy="0" iyz="0" ixz="0"/>
-    </xacro:macro>
-    <xacro:macro name="cylinder_inertia_def" params="radius length mass">
-    <inertia ixx="${mass * radius* radius / 2}"
-	     iyy="${mass * radius* radius / 2}"
-	     izz="${mass * (3 * radius * radius + length * length) / 12}"
-	     ixy="0" iyz="0" ixz="0"/>
-    </xacro:macro>
+  <xacro:include filename="$(find kuka_control)/urdf/definitions.xacro" />
     <xacro:macro name="tool" params="name parent *origin">
       <joint name="${name}_base_joint" type="fixed">
@@ -72,25 +59,42 @@
           <xacro:cylinder_inertia_def radius="0.005" length="0.01" mass="0.001"/>
         </inertial>
-        <visual>
+        <!--<visual>
           <origin xyz="0 0 0" rpy="0 0 0" />
           <geometry>
-            <mesh filename="package://kuka_control/models/tool/meshes/Tool_tip.dae"/>
+            <mesh filename="package://kuka_control/models/tool/meshes/Tool_tip.stl" scale="1 1 1"/>
           </geometry>
+          <material name="Aluminum"/>
+        </visual>-->
+        <visual>
+          <origin xyz="0 0 0.1" rpy="0 0 0" />
+          <geometry>
+            <cylinder length="0.02" radius="0.02"/>
+          </geometry>
+          <material name="Aluminum"/>
         </visual>
         <collision>
           <origin xyz="0 0 0" rpy="0 0 0" />
           <geometry>
-            <mesh filename="package://kuka_control/models/tool/meshes/Tool_tip.dae"/>
+            <mesh filename="package://kuka_control/models/tool/meshes/Tool_tip.stl" scale="1 1 1"/>
           </geometry>
         </collision>
       </link>
-      <gazebo reference="${name}_tip">
-        <turnGravityOff>true</turnGravityOff>
-        <selfCollide>true</selfCollide>
+      <!--<gazebo reference="${name}_tip">
+        <turnGravityOff>false</turnGravityOff>
+        <selfCollide>false</selfCollide>
         <mu1 value="1" />
         <mu2 value="1" />
-        <kp  value="1000000" />
-        <kd  value="0.1" />
-        <material>Gazebo/Grey</material>
+        <kp  value="100000" />
+        <kd  value="100.0" />
+        <material>aluminum</material>
+      </gazebo>-->
+      <gazebo reference="${name}_tip">
+        <turnGravityOff>false</turnGravityOff>
+        <selfCollide>false</selfCollide>
+        <mu1 value="0.1" />
+        <mu2 value="0.1" />
+        <kp  value="100000" />
+        <kd  value="1.0" />
+        <material>aluminum</material>
       </gazebo>
     </xacro:macro>

Commit message: Manfrotto model added. Launch and xacro files updated to be able to run real and simulated robot without conflict.

File: kuka_control/models/cell/cell.urdf.xacro (robot description, xacro)
@@ -5,5 +5,8 @@
   <xacro:include filename="$(find kuka_control)/models/cell/cell.xacro"/>
   <!-- Depth cameras -->
-  <xacro:include filename="$(find kuka_control)/models/sensors/camera.urdf.xacro" />
+<!--  <xacro:include filename="$(find kuka_control)/models/sensors/camera.urdf.xacro" />-->
+  <xacro:include filename="$(find kuka_control)/models/sensors/camera_manfrotto.urdf.xacro">
+  	<xacro:arg name="gazebo" value="$(arg gazebo)"/>
+  </xacro:include>
   <!-- Car door -->
 <!--  <xacro:include filename="$(find kuka_control)/models/car_door/car_door.urdf.xacro" />-->

File: kuka_control/models/sensors/asus_camera.urdf.xacro (robot description, xacro)
@@ -3,6 +3,6 @@
     <xacro:property name="M_PI" value="3.1415926535897931" />
     <!--
-     The asus_camera_model macro only adds the model, it does not also add
-     the openni gazebo plugin. See the 'asus_camera' macro below for that
+     The asus_camera macro only adds the model, it does not also add
+     the openni gazebo plugin. See the 'asus_camera_gazebo' macro below for that
     -->
     <xacro:macro name="asus_camera_model" params="name parent *origin">
@@ -68,9 +68,10 @@
      the openni gazebo plugin.
     -->
-    <xacro:macro name="asus_camera" params="name parent *origin">
+    <xacro:macro name="asus_camera" params="name parent gazebo *origin">
       <xacro:asus_camera_model name="${name}" parent="${parent}">
         <xacro:insert_block name="origin" />
       </xacro:asus_camera_model>
       <!-- ASUS Xtion PRO camera for simulation -->
+      <xacro:if value="${gazebo=='true'}">
       <gazebo reference="${name}_depth_frame">
         <sensor type="depth" name="${name}">
@@ -81,8 +82,8 @@
               <!--<format>R8G8B8</format>-->
               <format>B8G8R8</format>
-              <width>640</width>
-              <height>480</height>
-              <!--<width>320</width>
-              <height>240</height>-->
+              <!--<width>640</width>
+              <height>480</height>-->
+              <width>320</width>
+              <height>240</height>
             </image>
             <clip>
@@ -101,4 +102,5 @@
         </sensor>
       </gazebo>
+      </xacro:if>
     </xacro:macro>
   </robot>

File: kuka_control/models/sensors/camera.urdf.xacro (robot description, xacro)
@@ -6,13 +6,13 @@
   <xacro:include filename="$(find kuka_control)/models/sensors/kinect_camera.urdf.xacro" />
  <!--  Kinect sensor (k1) -->
-  <xacro:kinect_camera name="camera1" parent="cell_link">
+  <xacro:kinect_camera name="camera1" parent="cell_link" gazebo="$(arg gazebo)">
     <origin xyz="0.04 0.925 1.98" rpy="${-2*M_PI/180.0} ${58.0*M_PI/180.0} ${-M_PI/2+1*M_PI/180.0}" />
   </xacro:kinect_camera>
  <!--  Kinect sensor (k2) -->
-  <xacro:kinect_camera name="camera2" parent="cell_link">
+  <xacro:kinect_camera name="camera2" parent="cell_link" gazebo="$(arg gazebo)">
     <origin xyz="-0.04 -0.925 1.96" rpy="0 ${57.0*M_PI/180.0} ${M_PI/2.0+2*M_PI/180.0}" />
   </xacro:kinect_camera>
  <!--  Kinect sensor (k3) -->
-  <xacro:kinect_camera name="camera3" parent="cell_link">
+  <xacro:kinect_camera name="camera3" parent="cell_link" gazebo="$(arg gazebo)">
     <origin xyz="-1.2 0.95 1.05" rpy="${0.5*M_PI/180.0} ${5*M_PI/180.0} ${-65*M_PI/180.0}" />
   </xacro:kinect_camera>

File: kuka_control/models/sensors/camera_4kinects.urdf.xacro (robot description, xacro)
@@ -6,17 +6,17 @@
   <xacro:include filename="$(find kuka_control)/models/sensors/kinect_camera.urdf.xacro" />
   <!-- Kinect sensor (k1) -->
-  <xacro:kinect_camera name="camera1" parent="cell_link">
+  <xacro:kinect_camera name="camera1" parent="cell_link" gazebo="$(arg gazebo)">
       <origin xyz="-1.0 0.0 2.0" rpy="0 ${40.0*M_PI/180.0} 0" />
   </xacro:kinect_camera>
   <!-- Kinect sensor (k2) -->
-  <xacro:kinect_camera name="camera2" parent="cell_link">
+  <xacro:kinect_camera name="camera2" parent="cell_link" gazebo="$(arg gazebo)">
     <origin xyz="0.0 -1.0 2.0" rpy="0 ${40.0*M_PI/180.0} ${M_PI/2}" />
   </xacro:kinect_camera>
   <!-- Kinect sensor (k3) -->
-  <xacro:kinect_camera name="camera3" parent="cell_link">
+  <xacro:kinect_camera name="camera3" parent="cell_link" gazebo="$(arg gazebo)">
       <origin xyz="1.0 0.0 2.0" rpy="0 ${40.0*M_PI/180.0} ${M_PI}" />
   </xacro:kinect_camera>
   <!-- Kinect sensor (k4) -->
-  <xacro:kinect_camera name="camera4" parent="cell_link">
+  <xacro:kinect_camera name="camera4" parent="cell_link" gazebo="$(arg gazebo)">
     <origin xyz="0.0 1.0 2.0" rpy="0 ${40.0*M_PI/180.0} ${-M_PI/2.0}" />
   </xacro:kinect_camera>

File: kuka_control/models/sensors/kinect_camera.urdf.xacro (robot description, xacro)
@@ -52,9 +52,10 @@
       <link name="${name}_rgb_optical_frame"/>
     </xacro:macro>
-    <xacro:macro name="kinect_camera" params="name parent *origin">
+    <xacro:macro name="kinect_camera" params="name parent gazebo *origin">
       <xacro:kinect_camera_model name="${name}" parent="${parent}">
         <xacro:insert_block name="origin" />
       </xacro:kinect_camera_model>
-<!--
+      <!-- Kinect camera for simulation -->
+      <xacro:if value="${gazebo=='true'}">
       <gazebo reference="${name}_depth_frame">
         <sensor type="depth" name="${name}">
@@ -66,11 +67,11 @@
               <!--<width>640</width>
               <height>480</height>-->
-              <!--<width>320</width>
-              <height>240</height>-->
-           <!--   <width>160</width>
-              <height>120</height>
+              <width>320</width>
+              <height>240</height>
+              <!--<width>160</width>
+              <height>120</height>-->
             </image>
             <clip>
-              <near>0.05</near>
+              <near>0.5</near>
               <far>3</far>
             </clip>
@@ -85,5 +86,6 @@
           </plugin>
         </sensor>
-      </gazebo> -->
+      </gazebo>
+      </xacro:if>
     </xacro:macro>
   </robot>
