Commit message: pykdl updated. FT sensor issues improved but not solved

File: kuka_control/models/box/box.xacro (robot description, xacro)
@@ -30,5 +30,5 @@
   </joint>
   <gazebo reference="${name}_link">
-      <turnGravityOff>false</turnGravityOff>
+      <!--<turnGravityOff>false</turnGravityOff>-->
       <selfCollide>false</selfCollide>
       <!--<material>Gazebo/Red</material>-->

File: kuka_control/models/eraser/eraser.xacro (robot description, xacro)
@@ -32,5 +32,5 @@
   </link>
   <gazebo reference="${side}_velcro_base">
-    <turnGravityOff>true</turnGravityOff>
+    <!--<turnGravityOff>true</turnGravityOff>-->
     <selfCollide>true</selfCollide>
     <mu1 value="0.01" />
@@ -66,5 +66,5 @@
   </link>
   <gazebo reference="${side}_tool_base">
-    <turnGravityOff>true</turnGravityOff>
+    <!--<turnGravityOff>true</turnGravityOff>-->
     <selfCollide>true</selfCollide>
     <mu1 value="0.01" />
@@ -101,5 +101,5 @@
   </link>
   <gazebo reference="${side}_tool0">
-    <turnGravityOff>true</turnGravityOff>
+    <!--<turnGravityOff>true</turnGravityOff>-->
     <selfCollide>true</selfCollide>
     <mu1 value="0.01" />
@@ -136,5 +136,5 @@
   </link>
   <gazebo reference="${side}_tool_tip">
-    <turnGravityOff>true</turnGravityOff>
+    <!--<turnGravityOff>true</turnGravityOff>-->
     <selfCollide>true</selfCollide>
     <mu1 value="0.01" />

File: kuka_control/models/ft_sensor/ft_sensor_ati.gazebo.xacro (robot description, xacro)
@@ -11,17 +11,13 @@
       <provideFeedback>true</provideFeedback>
     </gazebo>
-    <!-- The ft_sensor plugin  -->
+    <!-- The ft_sensor plugin -->
     <gazebo>
-        <plugin name="${name}_ft_sensor" filename="libgazebo_ros_ft_sensor.so">
+      <plugin name="${name}_ft_sensor" filename="libgazebo_ros_ft_sensor.so">
         <updateRate>100.0</updateRate>
         <topicName>${name}/ft_sensor_topic</topicName>
         <jointName>${name}_measure_joint</jointName>
-        <noise>
-          <type>gaussian</type>
-          <mean>0.0</mean>
-          <stddev>0.0</stddev> <!-- change this to simulate noise -->
-        </noise>
-        </plugin>
-    </gazebo>
+        <gaussianNoise>0.001</gaussianNoise>
+      </plugin>
+	</gazebo>
     </xacro:macro>
 </robot>

File: kuka_control/models/ft_sensor/models.urdf.xacro (robot description, xacro)
@@ -10,8 +10,8 @@
 	</xacro:macro>
 	<xacro:macro name="cylinder_inertia_def" params="radius length mass">
-	<inertia ixx="${mass * radius* radius / 2}"
-		 iyy="${mass * radius* radius / 2}"
-		 izz="${mass * (3 * radius * radius + length * length) / 12}"
-		 ixy="0" iyz="0" ixz="0"/>
+	<inertia ixx="${mass * (3 * radius * radius + length * length) / 12}"
+		     iyy="${mass * (3 * radius * radius + length * length) / 12}"
+		     izz="${mass * radius* radius / 2}"
+		     ixy="0" iyz="0" ixz="0"/>
 	</xacro:macro>
 	<!-- ############# -->

File: kuka_control/models/ft_tool.xacro (robot description, xacro)
@@ -11,4 +11,9 @@
     <origin xyz="0 0 0.019" rpy="0 0 0"/>
   </xacro:ft_sensor_axia80>
+  <!-- Include the force-torque-sensor model -->
+  <!--<xacro:include filename="$(find sensor_description)/urdf/ft_sensor_ati.urdf.xacro"/>
+  <xacro:ft_sensor_ft45 parent="brida_link" name="axia80" type="ft45">
+    <origin xyz="0 0 0" rpy="0 0 0"/>
+  </xacro:ft_sensor_ft45>-->
   <!-- Include tool model -->
   <xacro:include filename="$(find kuka_control)/models/tool/tool.xacro"/>

File: kuka_control/models/tool/tool.xacro (robot description, xacro)
@@ -1,5 +1,19 @@
 <?xml version="1.0"?>
 <robot xmlns:xacro="http://ros.org/wiki/xacro">
-  <xacro:include filename="$(find kuka_control)/urdf/definitions.xacro" />
+  <!--<xacro:include filename="$(find kuka_control)/urdf/definitions.xacro" />-->
+  	<!-- Common tools: PI, inertias of a cuboid and cylinder -->
+	<xacro:property name="M_PI" value="3.1415926535897931"/>
+	<xacro:macro name="cuboid_inertia_def" params="width height length mass">
+	<inertia ixx="${mass * (height * height + length * length) / 12}"
+		     iyy="${mass * (width * width + length * length) / 12}"
+		     izz="${mass * (width * width + height * height) / 12}"
+		     ixy="0" iyz="0" ixz="0"/>
+	</xacro:macro>
+	<xacro:macro name="cylinder_inertia_def" params="radius length mass">
+	<inertia ixx="${mass * (3 * radius * radius + length * length) / 12}"
+		     iyy="${mass * (3 * radius * radius + length * length) / 12}"
+		     izz="${mass * radius* radius / 2}"
+		     ixy="0" iyz="0" ixz="0"/>
+	</xacro:macro>
     <xacro:macro name="tool" params="name parent *origin">
       <joint name="${name}_base_joint" type="fixed">
@@ -10,7 +24,7 @@
       <!--<link name="${name}_link">
         <inertial>
-          <mass value="0.1" />
-          <origin xyz="0 0 0" rpy="0 0 0" />
-          <inertia ixx="0.0001" ixy="0" ixz="0" iyy="0.0001" iyz="0" izz="0.0001" />
+          <mass value="0.2" />
+          <origin xyz="0 0 0.045" rpy="0 0 0" />
+          <xacro:cylinder_inertia_def radius="0.0325" length="0.09" mass="0.2"/>
         </inertial>
         <visual>
@@ -30,5 +44,5 @@
         <inertial>
           <mass value="0.2" />
-          <origin xyz="0 0 0" rpy="0 0 0" />
+          <origin xyz="0 0 0.045" rpy="0 0 0" />
           <!--<inertia ixx="0.0001" ixy="0" ixz="0" iyy="0.0001" iyz="0" izz="0.0001" />-->
           <xacro:cylinder_inertia_def radius="0.0325" length="0.09" mass="0.2"/>
@@ -55,9 +69,9 @@
         <inertial>
           <mass value="0.001" />
-          <origin xyz="0 0 0" rpy="0 0 0" />
+          <origin xyz="0 0 0.005" rpy="0 0 0" />
           <!--<inertia ixx="0.00001" ixy="0" ixz="0" iyy="0.00001" iyz="0" izz="0.00001" />-->
           <xacro:cylinder_inertia_def radius="0.005" length="0.01" mass="0.001"/>
         </inertial>
-        <!--<visual>
+        <visual>
           <origin xyz="0 0 0" rpy="0 0 0" />
           <geometry>
@@ -65,6 +79,6 @@
           </geometry>
           <material name="Aluminum"/>
-        </visual>-->
-        <visual>
+        </visual>
+        <!--<visual>
           <origin xyz="0 0 0.1" rpy="0 0 0" />
           <geometry>
@@ -72,5 +86,5 @@
           </geometry>
           <material name="Aluminum"/>
-        </visual>
+        </visual>-->
         <collision>
           <origin xyz="0 0 0" rpy="0 0 0" />
@@ -80,20 +94,12 @@
         </collision>
       </link>
-      <!--<gazebo reference="${name}_tip">
-        <turnGravityOff>false</turnGravityOff>
-        <selfCollide>false</selfCollide>
-        <mu1 value="1" />
-        <mu2 value="1" />
+      <gazebo reference="${name}_tip">
+        <!--<turnGravityOff>false</turnGravityOff>
+        <selfCollide>false</selfCollide>-->
+        <!--<mu1 value="0.1" />
+        <mu2 value="0.1" />-->
+        <mu value="0.1" />
         <kp  value="100000" />
-        <kd  value="100.0" />
-        <material>aluminum</material>
-      </gazebo>-->
-      <gazebo reference="${name}_tip">
-        <turnGravityOff>false</turnGravityOff>
-        <selfCollide>false</selfCollide>
-        <mu1 value="0.1" />
-        <mu2 value="0.1" />
-        <kp  value="100000" />
-        <kd  value="1.0" />
+        <kd  value="0.01" />
         <material>aluminum</material>
       </gazebo>

File: kuka_description/urdf/kr6r900sixx.gazebo.xacro (robot description, xacro)
@@ -17,4 +17,25 @@
     </plugin>
   </gazebo>
+<!-- Joint damping -->
+<!--
+  <gazebo reference="joint_a1">
+    <implicitSpringDamper>1</implicitSpringDamper>
+  </gazebo>
+  <gazebo reference="joint_a2">
+    <implicitSpringDamper>1</implicitSpringDamper>
+  </gazebo>
+  <gazebo reference="joint_a3">
+    <implicitSpringDamper>1</implicitSpringDamper>
+  </gazebo>
+  <gazebo reference="joint_a4">
+    <implicitSpringDamper>1</implicitSpringDamper>
+  </gazebo>
+  <gazebo reference="joint_a5">
+    <implicitSpringDamper>1</implicitSpringDamper>
+  </gazebo>
+  <gazebo reference="joint_a6">
+    <implicitSpringDamper>1</implicitSpringDamper>
+  </gazebo>
+-->
 <!--Transmission and actuators-->
   <transmission name="tran1">

File: kuka_description/urdf/kr6r900sixx_macro.xacro (robot description, xacro)
@@ -28,4 +28,6 @@
   <xacro:property name="diameter6" value="0.033" />
   <xacro:property name="max_effort" value="1200" />
+  <xacro:property name="damping" value="0.0"/>
+  <xacro:property name="friction" value="0.0"/>
   <xacro:macro name="kuka_kr6r900sixx" params="prefix">
     <link name="${prefix}base_link">
@@ -177,4 +179,5 @@
       <axis xyz="0 0 -1"/>
       <limit effort="${max_effort}" lower="${-DEG2RAD * 170}" upper="${DEG2RAD * 170}" velocity="${DEG2RAD * 300}"/>
+      <dynamics damping="${damping}" friction="${friction}"/>
     </joint>
     <joint name="${prefix}joint_a2" type="revolute">
@@ -184,4 +187,5 @@
       <axis xyz="0 1 0"/>
       <limit effort="${max_effort}" lower="${-DEG2RAD * 190}" upper="${DEG2RAD * 45}" velocity="${DEG2RAD * 225}"/>
+      <dynamics damping="${damping}" friction="${friction}"/>
     </joint>
     <joint name="${prefix}joint_a3" type="revolute">
@@ -191,4 +195,5 @@
       <axis xyz="0 1 0"/>
       <limit effort="${max_effort}" lower="${-DEG2RAD * 120}" upper="${DEG2RAD * 156}" velocity="${DEG2RAD * 225}"/>
+      <dynamics damping="${damping}" friction="${friction}"/>
     </joint>
     <joint name="${prefix}joint_a4" type="revolute">
@@ -198,4 +203,5 @@
       <axis xyz="-1 0 0"/>
       <limit effort="${max_effort}" lower="${-DEG2RAD * 185}" upper="${DEG2RAD * 185}" velocity="${DEG2RAD * 381}"/>
+      <dynamics damping="${damping}" friction="${friction}"/>
     </joint>
     <joint name="${prefix}joint_a5" type="revolute">
@@ -205,4 +211,5 @@
       <axis xyz="0 1 0"/>
       <limit effort="${max_effort}" lower="${-DEG2RAD * 120}" upper="${DEG2RAD * 120}" velocity="${DEG2RAD * 311}"/>
+      <dynamics damping="${damping}" friction="${friction}"/>
     </joint>
     <joint name="${prefix}joint_a6" type="revolute">
@@ -212,4 +219,5 @@
       <axis xyz="-1 0 0"/>
       <limit effort="${max_effort}" lower="${-DEG2RAD * 350}" upper="${DEG2RAD * 350}" velocity="${DEG2RAD * 492}"/>
+      <dynamics damping="${damping}" friction="${friction}"/>
     </joint>
     <joint name="${prefix}joint_a6-tool0" type="fixed">
