Commit message: launch and xacro files updated. Gamepad teleop node improved. Rviz modified to be used for polishing tests

File: kuka_control/models/box/box.urdf.xacro (robot description, xacro)
@@ -5,5 +5,5 @@
   <xacro:include filename="$(find kuka_control)/models/box/box.xacro"/>
   <!-- Box -->
-  <xacro:box_metal name="box" parent="base_link">
+  <xacro:box_metal name="box" parent="cell_link">
       <origin xyz="0.0 0.0 0.74" rpy="0 0 0" />
   </xacro:box_metal>

File: kuka_control/models/car_door/car_door.urdf.xacro (robot description, xacro)
@@ -5,5 +5,5 @@
   <xacro:include filename="$(find kuka_control)/models/car_door/car_door.xacro"/>
   <!-- Car door (Vito) -->
-  <xacro:car_door name="door1" parent="base_link">
+  <xacro:car_door name="door1" parent="cell_link">
       <origin xyz="0.0 0.0 0.8" rpy="0 0 0" />
   </xacro:car_door>

File: kuka_control/models/cell/cell.urdf.xacro (robot description, xacro)
@@ -8,4 +8,4 @@
   <!-- Car door -->
 <!--  <xacro:include filename="$(find kuka_control)/models/car_door/car_door.urdf.xacro" />-->
-  <xacro:include filename="$(find kuka_control)/models/box/box.urdf.xacro" />
+<!--  <xacro:include filename="$(find kuka_control)/models/box/box.urdf.xacro" />-->
 </robot>

File: kuka_control/models/cell/cell.xacro (robot description, xacro)
@@ -2,6 +2,6 @@
 <robot name="cell" xmlns:xacro="http://ros.org/wiki/xacro">
   <!-- World frame (for Gazebo) -->
-  <link name="world"/>
-  <link name="base_link">
+  <link name="cell/world"/>
+  <link name="cell_link">
       <inertial>
           <mass value="500" />
@@ -23,6 +23,6 @@
   <joint name="base_joint" type="fixed">
       <origin xyz="0.0 0.0 0.0" rpy="0 0 0" />
-      <parent link="world" />
-      <child link="base_link"/>
+      <parent link="cell/world" />
+      <child link="cell_link"/>
   </joint>
   <gazebo>

File: kuka_control/models/sensors/camera.urdf.xacro (robot description, xacro)
@@ -6,10 +6,14 @@
   <xacro:include filename="$(find kuka_control)/models/sensors/kinect_camera.urdf.xacro" />
  <!--  Kinect sensor (k1) -->
-  <xacro:kinect_camera name="camera1" parent="base_link">
+  <xacro:kinect_camera name="camera1" parent="cell_link">
     <origin xyz="0.04 0.925 1.98" rpy="${-2*M_PI/180.0} ${58.0*M_PI/180.0} ${-M_PI/2+1*M_PI/180.0}" />
   </xacro:kinect_camera>
  <!--  Kinect sensor (k2) -->
-  <xacro:kinect_camera name="camera2" parent="base_link">
+  <xacro:kinect_camera name="camera2" parent="cell_link">
     <origin xyz="-0.04 -0.925 1.96" rpy="0 ${57.0*M_PI/180.0} ${M_PI/2.0+2*M_PI/180.0}" />
   </xacro:kinect_camera>
+ <!--  Kinect sensor (k3) -->
+  <xacro:kinect_camera name="camera3" parent="cell_link">
+    <origin xyz="-1.2 0.95 1.05" rpy="${0.5*M_PI/180.0} ${5*M_PI/180.0} ${-65*M_PI/180.0}" />
+  </xacro:kinect_camera>
 </robot>

File: kuka_control/models/sensors/camera_4kinects.urdf.xacro (robot description, xacro)
@@ -6,17 +6,17 @@
   <xacro:include filename="$(find kuka_control)/models/sensors/kinect_camera.urdf.xacro" />
   <!-- Kinect sensor (k1) -->
-  <xacro:kinect_camera name="camera1" parent="base_link">
+  <xacro:kinect_camera name="camera1" parent="cell_link">
       <origin xyz="-1.0 0.0 2.0" rpy="0 ${40.0*M_PI/180.0} 0" />
   </xacro:kinect_camera>
   <!-- Kinect sensor (k2) -->
-  <xacro:kinect_camera name="camera2" parent="base_link">
+  <xacro:kinect_camera name="camera2" parent="cell_link">
     <origin xyz="0.0 -1.0 2.0" rpy="0 ${40.0*M_PI/180.0} ${M_PI/2}" />
   </xacro:kinect_camera>
   <!-- Kinect sensor (k3) -->
-  <xacro:kinect_camera name="camera3" parent="base_link">
+  <xacro:kinect_camera name="camera3" parent="cell_link">
       <origin xyz="1.0 0.0 2.0" rpy="0 ${40.0*M_PI/180.0} ${M_PI}" />
   </xacro:kinect_camera>
   <!-- Kinect sensor (k4) -->
-  <xacro:kinect_camera name="camera4" parent="base_link">
+  <xacro:kinect_camera name="camera4" parent="cell_link">
     <origin xyz="0.0 1.0 2.0" rpy="0 ${40.0*M_PI/180.0} ${-M_PI/2.0}" />
   </xacro:kinect_camera>
