Commit message: Roslaunch updated to work with real depth cameras. New parameter to enable/disable Gazebo simulation

File: kuka_control/models/sensors/camera.urdf.xacro (robot description, xacro)
@@ -5,19 +5,11 @@
   <xacro:include filename="$(find kuka_control)/models/sensors/asus_camera.urdf.xacro" />
   <xacro:include filename="$(find kuka_control)/models/sensors/kinect_camera.urdf.xacro" />
-  <!-- Kinect sensor (k1) -->
+ <!--  Kinect sensor (k1) -->
   <xacro:kinect_camera name="camera1" parent="base_link">
-      <origin xyz="-1.0 0.0 2.0" rpy="0 ${40.0*M_PI/180.0} 0" />
+    <origin xyz="0.0 1.0 2.0" rpy="0 ${30.0*M_PI/180.0} ${-M_PI/2}" />
   </xacro:kinect_camera>
-  <!-- Kinect sensor (k2) -->
+ <!--  Kinect sensor (k2) -->
   <xacro:kinect_camera name="camera2" parent="base_link">
-    <origin xyz="0.0 -1.0 2.0" rpy="0 ${40.0*M_PI/180.0} ${M_PI/2}" />
-  </xacro:kinect_camera>
-  <!-- Kinect sensor (k3) -->
-  <xacro:kinect_camera name="camera3" parent="base_link">
-      <origin xyz="1.0 0.0 2.0" rpy="0 ${40.0*M_PI/180.0} ${M_PI}" />
-  </xacro:kinect_camera>
-  <!-- Kinect sensor (k4) -->
-  <xacro:kinect_camera name="camera4" parent="base_link">
-    <origin xyz="0.0 1.0 2.0" rpy="0 ${40.0*M_PI/180.0} ${-M_PI/2.0}" />
+    <origin xyz="0.0 -1.0 2.0" rpy="0 ${30.0*M_PI/180.0} ${M_PI/2.0}" />
   </xacro:kinect_camera>
 </robot>

Commit message: URDF models and RViz configuration file adapted to real kinects

File: kuka_control/models/sensors/camera.urdf.xacro (robot description, xacro)
@@ -7,9 +7,9 @@
  <!--  Kinect sensor (k1) -->
   <xacro:kinect_camera name="camera1" parent="base_link">
-    <origin xyz="0.0 1.0 2.0" rpy="0 ${30.0*M_PI/180.0} ${-M_PI/2}" />
+    <origin xyz="0.04 0.925 1.98" rpy="${-2*M_PI/180.0} ${58.0*M_PI/180.0} ${-M_PI/2+1*M_PI/180.0}" />
   </xacro:kinect_camera>
  <!--  Kinect sensor (k2) -->
   <xacro:kinect_camera name="camera2" parent="base_link">
-    <origin xyz="0.0 -1.0 2.0" rpy="0 ${30.0*M_PI/180.0} ${M_PI/2.0}" />
+    <origin xyz="-0.04 -0.925 1.96" rpy="0 ${57.0*M_PI/180.0} ${M_PI/2.0+2*M_PI/180.0}" />
   </xacro:kinect_camera>
 </robot>

File: kuka_control/models/sensors/kinect_camera.urdf.xacro (robot description, xacro)
@@ -56,4 +56,5 @@
         <xacro:insert_block name="origin" />
       </xacro:kinect_camera_model>
+<!--
       <gazebo reference="${name}_depth_frame">
         <sensor type="depth" name="${name}">
@@ -62,10 +63,10 @@
             <horizontal_fov>${60 * M_PI/180.0}</horizontal_fov>
             <image>
-              <format>B8G8R8</format>
+              <format>B8G8R8</format>-->
               <!--<width>640</width>
               <height>480</height>-->
               <!--<width>320</width>
               <height>240</height>-->
-              <width>160</width>
+           <!--   <width>160</width>
               <height>120</height>
             </image>
@@ -84,5 +85,5 @@
           </plugin>
         </sensor>
-      </gazebo>
+      </gazebo> -->
     </xacro:macro>
   </robot>
